Commit message: feat: Spot 전환 + 2-카메라 + C2 웹 브리지 완성 + 개발문서 체계 구축
## 주요 변경

### Main PC (Isaac Sim)
- spot_with_arm → Spot (12-DOF, SpotFlatTerrainPolicy) 전환
- 단일 손목카메라 → 전/후방 기체 카메라 2개 (OmniGraph 이중 파이프라인)
- video_degrade_node: 하드코딩 토픽 → DEGRADE_IN/DEGRADE_OUT 환경변수
- run_degrade.sh: front+rear 2인스턴스 병렬 실행
- URDF: arm 링크/관절 제거 → 13링크 12관절

### C2 PC (FastAPI + Next.js)
- ros_bridge: 이중 카메라 구독, odom yaw 추출, arm_q 제거
- config: video 단일 → video_front/video_rear, CORS 기본값 "*"
- api.ts: API_BASE 모듈 상수 → getApiBase() 런타임 함수 (Next.js SSR 고정 버그 수정)
- VideoWall: WebRTC+MJPEG 폴백, getApiBase() 사용
- SpotSurroundView: Three.js 3D 로봇 뷰 (yaw 폴링, 전후방 frustum, 커버리지 링)
- debug 페이지: SpotSurroundView + Lichtblick iframe
- uvicorn[standard]+websockets 필수 (WS /events 지원)
- Lichtblick layout: 전/후방 카메라 이중 패널

### 개발문서
- dev-docs/ 7개 문서 신규 (README, architecture, main-side, sub1-side,
  ros2-interface, ops, CHANGELOG)
- CLAUDE.md: source→doc 매핑 + 자동 갱신 규칙

Co-Authored-By: Claude Sonnet 4.6 <noreply@anthropic.com>

File: main_side/spot_isaac.urdf (robot description, URDF)
Before this commit: robot spot_with_arm, 20 links, 19 joints
Links:
- removed link arm0_link_el0
- removed link arm0_link_el1
- removed link arm0_link_fngr
- removed link arm0_link_sh0
- removed link arm0_link_sh1
- removed link arm0_link_wr0
- removed link arm0_link_wr1
- link base: geometry visual mesh filename=package://spot_description/meshes/base_simple/visual/body.o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
Joints:
- removed joint arm0_el0
- removed joint arm0_el1
- removed joint arm0_f1x
- removed joint arm0_sh0
- removed joint arm0_sh1
- removed joint arm0_wr0
- removed joint arm0_wr1
